File: hardware/kiCad/Mercury/Mercury.sch (KiCad schematic (older format))
At the start: 75 parts, among them J1 SWD, J10 OUTPUT, J11 Analog I/O, J12 Power Rails, J2 I2C1, J3 I2C2, J4 I2C1, J5 SPI1, J6 SPI2, J7 629105150521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

Commit message: Layout Begins
Parts:
- removed J2, J4: I2C1, Connector_Wire:SolderWire-0.25sqmm_1x04_P4.2mm_D0.65mm_OD1.7mm, symbol Connector_Generic:Conn_01x04
- removed J3: I2C2, Connector_Wire:SolderWire-0.25sqmm_1x04_P4.2mm_D0.65mm_OD1.7mm, symbol Connector_Generic:Conn_01x06
- removed J5: SPI1, Connector_Wire:SolderWire-0.25sqmm_1x05_P4.5mm_D0.65mm_OD2mm, symbol Connector_Generic:Conn_01x06
- removed J6: SPI2, Connector_Wire:SolderWire-0.25sqmm_1x05_P4.5mm_D0.65mm_OD2mm, symbol Connector_Generic:Conn_01x06
- added J2, J4: UART1, Connector_Wire:SolderWire-0.1sqmm_1x02_P3.6mm_D0.4mm_OD1mm, symbol Connector_Generic:Conn_01x02
- added J3: I2C2, Connector_Wire:SolderWire-0.1sqmm_1x04_P3.6mm_D0.4mm_OD1mm_Relief, symbol Connector_Generic:Conn_01x04
- added J5: SPI1, Connector_Wire:SolderWire-0.1sqmm_1x04_P3.6mm_D0.4mm_OD1mm, symbol Connector_Generic:Conn_01x04
- added J6: SPI2, Connector_Wire:SolderWire-0.1sqmm_1x04_P3.6mm_D0.4mm_OD1mm, symbol Connector_Generic:Conn_01x04
- C2, C3, C4, C5, C6, C7, C8: footprint Capacitor_SMD:C_0603_1608Metric -> Capacitor_SMD:C_0402_1005Metric
Connections:
- net +3V3: now also J12.2 (Pin_2); no longer J12.1 (Pin_1)
- net +5V: now also J12.1 (Pin_1); no longer J12.2 (Pin_2)
- net Input1: now also J9.3 (Pin_3); no longer J9.1 (Pin_1)
- net Input3: now also J9.1 (Pin_1); no longer J9.3 (Pin_3)
- net UART1_RX: now also U1.24 (PA1); no longer U1.69 (PA10)
- net UART1_TX: now also U1.23 (PA0); no longer U1.68 (PA9)
- net at R6.2: now also J3.1 (Pin_1)
- net at R7.2: now also J3.2 (Pin_2)
- net at R8.2: now also J3.3 (Pin_3)
- net at R9.2: now also J3.4 (Pin_4)
- net at R4.2: now also J2.1 (Pin_1)
- net at R5.2: now also J2.2 (Pin_2)
- net at R15.2: now also J4.2 (Pin_2)
- net at R14.2: now also J4.1 (Pin_1)
- net at R16.2: now also J5.1 (Pin_1)
- net at R17.2: now also J5.2 (Pin_2)
- net at R18.2: now also J5.3 (Pin_3)
- net at R19.2: now also J5.4 (Pin_4)
- net at R20.2: now also J6.1 (Pin_1)
- net at R21.2: now also J6.2 (Pin_2)
- net at R22.2: now also J6.3 (Pin_3)
- net at R23.2: now also J6.4 (Pin_4)
Other:
- moved on the sheet: C12
